Commit message: Mount the UR20 on the right side and the wrist camera along the gripper
The arm bracket was measured from the vehicle CAD: the UR20 sits on the
right (-y) side wall at (-0.006, -0.42, 0.881) with its z axis along -y. The
URDF had it 1.62 m away on the left. The bracket is added as its own link,
and the SRDF pairs between arm and vehicle that assumed the old mount are
checked again.

The ZED X looked sideways from the wrist. It now sits on a generic stand-in
bracket, 0.085 m off the tool axis and tilted 15 degrees toward the gripper,
with a wrist_camera collision link. The same numbers are in the scene patch,
the URDF and the scan controller's camera offset.

patch_scene_for_pruning.py applies both mounts, adds the arm bracket as a
visual and spawns the robot facing -x so the arm side faces the row. The
mission parks 1.65 m from the trunk, which keeps the same wheel clearance
as before, and 0.35 m behind it along the row, which keeps the scan clear
of the shoulder singularity for base yaw within 10 degrees. It also stops
the base when interrupted.

The scene, the vendored ZED X asset and the bracket mesh are added to DVC.

File: oskar_simulation/tipard_ur20_combined/tipard_ur20_combined.urdf (robot description, URDF)
Before this commit: robot tipard_ur20_combined, 31 links, 30 joints
Links:
- added link ur20_bracket; collision mesh filename=package://tipard_ur20_combined/meshes/ur20_bracket/ur20_bra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; visual mesh filename=package://tipard_ur20_combined/meshes/ur20_bracket/ur20_bra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
- added link wrist_camera; collision box size=0.028 0.05 0.016; collision box size=0.164 0.047 0.032
Joints:
- added joint tipard_to_ur20_bracket_joint: type fixed, parent base_link, child ur20_bracket, origin xyz=0 0 0 rpy=0 0 0
- added joint wrist_3_to_camera_joint: type fixed, parent wrist_3_link, child wrist_camera, origin xyz=0 0 0 rpy=0 0 0
- joint tipard_to_ur20_mount_joint: origin xyz=0.0 1.2 0.7 rpy=-1.5708 1.5708 0 -> xyz=-0.006 -0.42 0.881 rpy=1.5708 1.5708 0
